File: hardware/logger.sch (EAGLE design)
At the start: 40 parts, among them J1 MICRO_USB_B_HIROSE_ZX62-B-5PA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, SW1 TVAF06-A020B-R, U2 NJM12888F, X1 FA-238

Commit message: べたGND前です。esp32のschはノータッチなのでここに上がってないです。よろしくお願いします。
Connections:
- net VDD: now also RP1.RUN
Changed lines of the file:
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@@
 <segment>
 <pinref part="RP1" gate="G$1" pin="VREG_VIN"/>
-<wire x1="33.02" y1="127" x2="10.16" y2="127" width="0.1524" layer="91"/>
+<wire x1="33.02" y1="127" x2="30.48" y2="127" width="0.1524" layer="91"/>
 <pinref part="C3" gate="G$1" pin="1"/>
+<wire x1="30.48" y1="127" x2="10.16" y2="127" width="0.1524" layer="91"/>
 <wire x1="10.16" y1="127" x2="10.16" y2="124.46" width="0.1524" layer="91"/>
 <wire x1="10.16" y1="127" x2="10.16" y2="129.54" width="0.1524" layer="91"/>
 <junction x="10.16" y="127"/>
 <pinref part="VDD8" gate="G$1" pin="VDD"/>
+<pinref part="RP1" gate="G$1" pin="RUN"/>
+<wire x1="33.02" y1="121.92" x2="30.48" y2="121.92" width="0.1524" layer="91"/>
+<wire x1="30.48" y1="121.92" x2="30.48" y2="127" width="0.1524" layer="91"/>
+<junction x="30.48" y="127"/>
 </segment>
 <segment>

Commit message: シルクを調整
Parts:
- renumbered BT1 to BAT, MICROSD to MICRO_SD, U$1 to U1
Changed lines of the file:
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@@
 <part name="BOTTOM" library="pins" deviceset="P5_2.54" device=""/>
 <part name="U$2" library="pins" deviceset="P2_2_2.54" device=""/>
-<part name="MICROSD" library="dm3at-sf-pejm5" deviceset="DM3AT-SF-PEJM5" device=""/>
+<part name="MICRO_SD" library="dm3at-sf-pejm5" deviceset="DM3AT-SF-PEJM5" device=""/>
 <part name="GND1" library="supply1" library_urn="urn:adsk.eagle:library:371" deviceset="GND" device=""/>
 <part name="VDD1" library="supply1" library_urn="urn:adsk.eagle:library:371" deviceset="VDD" device=""/>
@@
 <part name="C16" library="rcl" library_urn="urn:adsk.eagle:library:334" deviceset="C-EU" device="C0402" package3d_urn="urn:adsk.eagle:package:23626/2"/>
 <part name="GND3" library="supply1" library_urn="urn:adsk.eagle:library:371" deviceset="GND" device=""/>
-<part name="BT1" library="MS414GE-FL26E" deviceset="MS414GE-FL26E" device=""/>
-<part name="U$1" library="rtc" deviceset="RX-8035LC" device="" package3d_urn="urn:adsk.eagle:package:37886091/1"/>
+<part name="BAT" library="MS414GE-FL26E" deviceset="MS414GE-FL26E" device=""/>
+<part name="U1" library="rtc" deviceset="RX-8035LC" device="" package3d_urn="urn:adsk.eagle:package:37886091/1"/>
 <part name="GND4" library="supply1" library_urn="urn:adsk.eagle:library:371" deviceset="GND" device=""/>
 <part name="VDD3" library="supply1" library_urn="urn:adsk.eagle:library:371" deviceset="VDD" device=""/>
@@
 <attribute name="VALUE" x="-5.08" y="144.78" size="1.778" layer="96"/>
 </instance>
-<instance part="MICROSD" gate="G$1" x="228.6" y="78.74" smashed="yes">
+<instance part="MICRO_SD" gate="G$1" x="228.6" y="78.74" smashed="yes">
 <attribute name="NAME" x="220.98" y="97.0548" size="2.54433125" layer="95"/>
 <attribute name="VALUE" x="220.98" y="57.8862" size="2.54358125" layer="96"/>
@@
 <attribute name="VALUE" x="177.8" y="-15.24" size="1.778" layer="96"/>
 </instance>
-<instance part="BT1" gate="G$1" x="195.58" y="127" smashed="yes" rot="R270">
+<instance part="BAT" gate="G$1" x="195.58" y="127" smashed="yes" rot="R270">
 <attribute name="NAME" x="199.39" y="130.81" size="1.778" layer="95" rot="R270"/>
 <attribute name="VALUE" x="190.5" y="130.81" size="1.778" layer="96" rot="R270"/>
 </instance>
-<instance part="U$1" gate="G$1" x="220.98" y="132.08" smashed="yes">
+<instance part="U1" gate="G$1" x="220.98" y="132.08" smashed="yes">
 <attribute name="NAME" x="210.82" y="144.78" size="1.778" layer="95"/>
 <attribute name="VALUE" x="210.82" y="114.3" size="1.778" layer="96"/>
@@
 </segment>
 <segment>
-<pinref part="MICROSD" gate="G$1" pin="A"/>
+<pinref part="MICRO_SD" gate="G$1" pin="A"/>
 <wire x1="215.9" y1="66.04" x2="193.04" y2="66.04" width="0.1524" layer="91"/>
 <wire x1="193.04" y1="66.04" x2="193.04" y2="60.96" width="0.1524" layer="91"/>
 <pinref part="GND1" gate="1" pin="GND"/>
-<pinref part="MICROSD" gate="G$1" pin="VSS"/>
+<pinref part="MICRO_SD" gate="G$1" pin="VSS"/>
 <wire x1="215.9" y1="76.2" x2="193.04" y2="76.2" width="0.1524" layer="91"/>
 <wire x1="193.04" y1="76.2" x2="193.04" y2="71.12" width="0.1524" layer="91"/>
@@
 <wire x1="193.04" y1="81.28" x2="193.04" y2="76.2" width="0.1524" layer="91"/>
 <junction x="193.04" y="76.2"/>
-<pinref part="MICROSD" gate="G$1" pin="SHIELD"/>
+<pinref part="MICRO_SD" gate="G$1" pin="SHIELD"/>
 <wire x1="215.9" y1="71.12" x2="193.04" y2="71.12" width="0.1524" layer="91"/>
 <junction x="193.04" y="71.12"/>
@@
 <pinref part="GND4" gate="1" pin="GND"/>
 <wire x1="203.2" y1="116.84" x2="203.2" y2="119.38" width="0.1524" layer="91"/>
-<pinref part="U$1" gate="G$1" pin="GND"/>
+<pinref part="U1" gate="G$1" pin="GND"/>
 <wire x1="203.2" y1="119.38" x2="208.28" y2="119.38" width="0.1524" layer="91"/>
-<pinref part="BT1" gate="G$1" pin="-"/>
+<pinref part="BAT" gate="G$1" pin="-"/>
 <wire x1="203.2" y1="119.38" x2="195.58" y2="119.38" width="0.1524" layer="91"/>
 <junction x="203.2" y="119.38"/>
@@
 </segment>
 <segment>
-<pinref part="MICROSD" gate="G$1" pin="VDD"/>
+<pinref part="MICRO_SD" gate="G$1" pin="VDD"/>
 <wire x1="215.9" y1="93.98" x2="193.04" y2="93.98" width="0.1524" layer="91"/>
 <wire x1="193.04" y1="93.98" x2="193.04" y2="96.52" width="0.1524" layer="91"/>
@@
 </segment>
 <segment>
-<pinref part="U$1" gate="G$1" pin="VDD"/>
+<pinref part="U1" gate="G$1" pin="VDD"/>
 <wire x1="185.42" y1="142.24" x2="208.28" y2="142.24" width="0.1524" layer="91"/>
 <wire x1="185.42" y1="142.24" x2="185.42" y2="144.78" width="0.1524" layer="91"/>
@@
 </segment>
 <segment>
-<pinref part="MICROSD" gate="G$1" pin="DAT0"/>
+<pinref part="MICRO_SD" gate="G$1" pin="DAT0"/>
 <wire x1="215.9" y1="91.44" x2="213.36" y2="91.44" width="0.1524" layer="91"/>
 <label x="213.36" y="91.44" size="1.778" layer="95" rot="R180" xref="yes"/>
@@
 </segment>
 <segment>
-<pinref part="MICROSD" gate="G$1" pin="CD/DAT3"/>
+<pinref part="MICRO_SD" gate="G$1" pin="CD/DAT3"/>
 <wire x1="215.9" y1="83.82" x2="213.36" y2="83.82" width="0.1524" layer="91"/>
 <label x="213.36" y="83.82" size="1.778" layer="95" rot="R180" xref="yes"/>
@@
 </segment>
 <segment>
-<pinref part="MICROSD" gate="G$1" pin="CLK"/>
+<pinref part="MICRO_SD" gate="G$1" pin="CLK"/>
 <wire x1="215.9" y1="78.74" x2="213.36" y2="78.74" width="0.1524" layer="91"/>
 <label x="213.36" y="78.74" size="1.778" layer="95" rot="R180" xref="yes"/>
@@
 </segment>
 <segment>
-<pinref part="MICROSD" gate="G$1" pin="CMD"/>
+<pinref part="MICRO_SD" gate="G$1" pin="CMD"/>
 <wire x1="215.9" y1="81.28" x2="213.36" y2="81.28" width="0.1524" layer="91"/>
 <label x="213.36" y="81.28" size="1.778" layer="95" rot="R180" xref="yes"/>
@@
 </segment>
 <segment>
-<pinref part="U$1" gate="G$1" pin="SDA"/>
+<pinref part="U1" gate="G$1" pin="SDA"/>
 <wire x1="233.68" y1="134.62" x2="236.22" y2="134.62" width="0.1524" layer="91"/>
 <label x="236.22" y="134.62" size="1.778" layer="95" xref="yes"/>
@@
 </segment>
 <segment>
-<pinref part="U$1" gate="G$1" pin="SCL"/>
+<pinref part="U1" gate="G$1" pin="SCL"/>
 <wire x1="233.68" y1="137.16" x2="236.22" y2="137.16" width="0.1524" layer="91"/>
 <label x="236.22" y="137.16" size="1.778" layer="95" xref="yes"/>
@@
 <net name="SD" class="0">
 <segment>
-<pinref part="MICROSD" gate="G$1" pin="B"/>
+<pinref part="MICRO_SD" gate="G$1" pin="B"/>
 <wire x1="215.9" y1="63.5" x2="213.36" y2="63.5" width="0.1524" layer="91"/>
 <label x="213.36" y="63.5" size="1.778" layer="95" rot="R180" xref="yes"/>
@@
 <net name="N$1" class="0">
 <segment>
-<pinref part="BT1" gate="G$1" pin="+"/>
-<pinref part="U$1" gate="G$1" pin="VBAT"/>
+<pinref part="BAT" gate="G$1" pin="+"/>
+<pinref part="U1" gate="G$1" pin="VBAT"/>
 <wire x1="195.58" y1="134.62" x2="203.2" y2="134.62" width="0.1524" layer="91"/>
-<pinref part="U$1" gate="G$1" pin="VOUT"/>
+<pinref part="U1" gate="G$1" pin="VOUT"/>
 <wire x1="203.2" y1="134.62" x2="208.28" y2="134.62" width="0.1524" layer="91"/>
 <wire x1="208.28" y1="137.16" x2="203.2" y2="137.16" width="0.1524" layer="91"/>

Commit message: 若干修正
Connections:
- removed net PWM5_B: RP1.GPIO11
- net SD: now also RP1.GPIO11
Changed lines of the file:
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@@
-</segment>
-</net>
-<net name="PWM5_B" class="0">
-<segment>
-<pinref part="RP1" gate="G$1" pin="GPIO11"/>
-<wire x1="33.02" y1="68.58" x2="30.48" y2="68.58" width="0.1524" layer="91"/>
-<label x="30.48" y="68.58" size="1.778" layer="95" rot="R180" xref="yes"/>
 </segment>
 </net>
@@
 <label x="213.36" y="63.5" size="1.778" layer="95" rot="R180" xref="yes"/>
 </segment>
+<segment>
+<pinref part="RP1" gate="G$1" pin="GPIO11"/>
+<wire x1="33.02" y1="68.58" x2="30.48" y2="68.58" width="0.1524" layer="91"/>
+<label x="30.48" y="68.58" size="1.778" layer="95" rot="R180" xref="yes"/>
+</segment>
 </net>
