File: hardware/esp32cam.brd (EAGLE design)
At the start: 33.5 x 34.6 mm, 46 parts, among them J1 MICRO_USB_B_HIROSE_ZX62-B-5PA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, Q1 HN1C01FU, U1 NJM11100, U2 NJM11100, U4 NJM12888F, U6 SPU0414HR5H-SB

Commit message: ベタ・シルク調整
Routing:
- net GND: vias 25 -> 120
